File: Robot1/robot1/robot1.kicad_pcb (KiCad board)
At the start: 2 copper layers, 6 parts

Commit message: Robot1 evolutions
Parts:
- removed the ? at (67.3, 125.7)
- added ?: , ben:Pin, F.Cu at (109.2, 182.9)
- added ?: , ben:Pin, F.Cu at (106.7, 182.9)
- added ?: , ben:Pin, F.Cu at (104.1, 182.9)
- added ?: , ben:Pin, F.Cu at (101.6, 182.9)
- added ?: , ben:Pin, F.Cu at (99.1, 182.9)
- added ?: , ben:Pin, F.Cu at (96.5, 182.9)
- added ?: , ben:Pin, F.Cu at (94.0, 182.9)
- added ?: , ben:Pin, F.Cu at (91.4, 182.9)
- added ?: , ben:Pin, F.Cu at (88.9, 182.9)
- added ?: , ben:Pin, F.Cu at (86.4, 182.9)
- added ?: , ben:Pin, F.Cu at (83.8, 182.9)
- added ?: , ben:Pin, F.Cu at (81.3, 182.9)
- added ?: , ben:Pin, F.Cu at (78.7, 182.9)
- added ?: Bornier3, ben:Bornier3, F.Cu at (68.6, 127.0)
- added ?: Condo, ben:Condo, F.Cu at (68.6, 146.1)
- added ?: Diode, ben:Diode, F.Cu at (78.7, 127.0)
- added ?: , ben:Pin, F.Cu at (66.0, 129.5)
- added ?: , ben:Pin, F.Cu at (66.0, 132.1)
- moved ? 48.4 mm to (114.3, 124.5)
- moved ? 25.0 mm to (104.1, 124.5)
- moved ? 21.6 mm to (86.4, 121.9)
- moved ? 1.80 mm to (91.4, 149.9)
- moved ? 1.27 mm to (91.4, 182.9)
